Commit message: [Feat]逐点规划成功

File: src/kuka_urdf/urdf/kuka_urdf.urdf (robot description, URDF)
Before this commit: robot kuka_urdf, 8 links, 7 joints
Links:
- added link link7, mass 0.0603242087036552; collision mesh filename=package://kuka_urdf/meshes/link7.STL; visual mesh filename=package://kuka_urdf/meshes/link7.STL
- link link1: mass 24.868772466875 -> 24.869
- link link2: mass 13.9287878174792 -> 13.929
- link link3: mass 16.4189284998869 -> 16.419
- link link5: mass 1.80204110195789 -> 1.73399119088313
Joints:
- added joint joint7: type fixed, parent link6, child link7, origin xyz=0 0.10377 0 rpy=-0.019531 0.017968 1.4875, axis 0 0 0
- joint joint1: type revolute -> continuous
- joint joint2: origin xyz=0.285000000000002 0.278999999999999 0 rpy=0 0 0.860540949726414 -> xyz=0.285 0.279 0 rpy=0 0 0.86054
- joint joint3: origin xyz=0 0.680000000000002 0 rpy=-3.14159265358979 0 2.25375212776307 -> xyz=0 0.68 0 rpy=-3.1416 0 2.2538
- joint joint4: origin xyz=-0.463043248331428 -0.0225000000000002 0.0330000000000008 rpy=3.14159265358979 -1.03989491708518 -1.57079632679491 -> xyz=-0.46304 -0.0225 0.033 rpy=3.1416 -1.0399 -1.5708; type revolute -> continuous
- joint joint5: origin xyz=0 0.203456751668462 0 rpy=1.69866961467948 0 -3.14159265358972 -> xyz=0 0.20346 0 rpy=1.6987 0 -3.1416
- joint joint6: origin xyz=-0.0160000000004577 0 0.185308798192681 rpy=1.57079632679489 0 2.12309994244728 -> xyz=-0.016 0 0.18531 rpy=1.5708 0 2.1231; type revolute -> continuous

Commit message: [Feat]加入转台

File: src/kuka_urdf/urdf/kuka_urdf.urdf (robot description, URDF)
Before this commit: robot kuka_urdf, 9 links, 8 joints
Links:
- added link tabelLink1, mass 0.060324; collision mesh filename=package://kuka_urdf/meshes/tabelLink1.STL; visual mesh filename=package://kuka_urdf/meshes/tabelLink1.STL
- added link tableBase, mass 22.655; collision mesh filename=package://kuka_urdf/meshes/tableBase.STL; visual mesh filename=package://kuka_urdf/meshes/tableBase.STL
- added link tableEeffortLink, mass 0.060324; collision mesh filename=package://kuka_urdf/meshes/tableEeffortLink.STL; visual mesh filename=package://kuka_urdf/meshes/tableEeffortLink.STL
- added link tableLink2, mass 0.32268; collision mesh filename=package://kuka_urdf/meshes/tableLink2.STL; visual mesh filename=package://kuka_urdf/meshes/tableLink2.STL
- link base_link: mass 72.8456791935468 -> 72.846
- link link1: mass 24.869 -> 0.060324
- link link2: mass 13.929 -> 0.060324
- link link3: mass 16.419 -> 0.060324
- link link4: mass 2.38078194379471 -> 0.060324
- link link5: mass 1.73399119088313 -> 0.060324
- link link6: mass 0.21569144856326 -> 0.060324
- link link7: mass 0.0603242087036552 -> 0.060324
Joints:
- added joint tableEeffortJoint: type fixed, parent tableLink2, child tableEeffortLink, origin xyz=0 0 0 rpy=1.5708 0 0, axis 0 0 0
- added joint tableJoint1: type continuous, parent tableBase, child tabelLink1, origin xyz=0 0 0 rpy=0 0 0, axis 0 0 1
- added joint tableJoint2: type continuous, parent tabelLink1, child tableLink2, origin xyz=0 0.116 0 rpy=-1.5708 0 0, axis 0 0 1
- added joint tableJointBase: type fixed, parent base_link, child tableBase, origin xyz=1 -0.01 0.21 rpy=1.5708 0 0, axis 0 0 0
- joint joint1: origin xyz=0 0 0.357 rpy=1.5707963267949 0 -0.0844304651404737 -> xyz=0 -0.00999999999999998 0.367 rpy=1.5707963267949 0 -0.0844304651404737
- joint joint2: origin xyz=0.285 0.279 0 rpy=0 0 0.86054 -> xyz=0.2751402982579 0.270669215850882 0 rpy=0 0 1.09776733459367; type revolute -> continuous
- joint joint3: origin xyz=0 0.68 0 rpy=-3.1416 0 2.2538 -> xyz=0.00300600653973404 0.670462499033651 0 rpy=3.14159265358979 0 2.17118981711903; type revolute -> continuous
- joint joint4: origin xyz=-0.46304 -0.0225 0.033 rpy=3.1416 -1.0399 -1.5708 -> xyz=-0.44629918087112 -0.0224999999999995 0.032999999999999 rpy=3.14159265358979 1.28637430236672 -1.5707963267949
- joint joint5: origin xyz=0 0.20346 0 rpy=1.6987 0 -3.1416 -> xyz=0 0.220200819128881 0 rpy=1.50631561095374 0 -3.14159265358979; type revolute -> continuous
- joint joint6: origin xyz=-0.016 0 0.18531 rpy=1.5708 0 2.1231 -> xyz=-0.0159999999999904 0 0.161511009128483 rpy=1.5707963267949 0 -0.91580856418439
- joint joint7: origin xyz=0 0.10377 0 rpy=-0.019531 0.017968 1.4875 -> xyz=0 0.0343289908715182 0 rpy=-3.14159265358978 -1.24624974571635 3.14159265358977

Commit message: [Feat]更换转台半球

File: src/kuka_urdf/urdf/kuka_urdf.urdf (robot description, URDF)
Before this commit: robot kuka_urdf, 13 links, 12 joints
Links:
- link base_link: mass 72.846 -> 72.8456791935468
- link link1: mass 0.060324 -> 15.0345564818104
- link link2: mass 0.060324 -> 13.9287847526223
- link link3: mass 0.060324 -> 12.8506822129936
- link link4: mass 0.060324 -> 2.38079247091277
- link link5: mass 0.060324 -> 1.73398183318851
- link link6: mass 0.060324 -> 0.21569146659832
- link link7: mass 0.060324 -> 0.0603242087036552
- link tabelLink1: mass 0.060324 -> 7.28336977784291
- link tableBase: mass 22.655 -> 22.6545515868041
- link tableEeffortLink: mass 0.060324 -> 3.48926224058707
- link tableLink2: mass 0.32268 -> 0.32267569246235
Joints:
- joint joint1: origin xyz=0 -0.00999999999999998 0.367 rpy=1.5707963267949 0 -0.0844304651404737 -> xyz=0 -0.01 0.367 rpy=1.5708 0 -0.08443
- joint joint2: origin xyz=0.2751402982579 0.270669215850882 0 rpy=0 0 1.09776733459367 -> xyz=0.27514 0.27067 0 rpy=0 0 1.0978
- joint joint3: origin xyz=0.00300600653973404 0.670462499033651 0 rpy=3.14159265358979 0 2.17118981711903 -> xyz=0.003006 0.67046 0 rpy=3.1416 0 2.1712
- joint joint4: origin xyz=-0.44629918087112 -0.0224999999999995 0.032999999999999 rpy=3.14159265358979 1.28637430236672 -1.5707963267949 -> xyz=-0.4463 -0.0225 0.033 rpy=3.1416 1.2864 -1.5708
- joint joint5: origin xyz=0 0.220200819128881 0 rpy=1.50631561095374 0 -3.14159265358979 -> xyz=0 0.2202 0 rpy=1.5063 0 -3.1416
- joint joint6: origin xyz=-0.0159999999999904 0 0.161511009128483 rpy=1.5707963267949 0 -0.91580856418439 -> xyz=-0.016 0 0.16151 rpy=1.5708 0 -0.91581
- joint joint7: origin xyz=0 0.0343289908715182 0 rpy=-3.14159265358978 -1.24624974571635 3.14159265358977 -> xyz=0 0.14433 0 rpy=-3.1416 -1.2462 3.1416
- joint tableEeffortJoint: origin xyz=0 0 0 rpy=1.5708 0 0 -> xyz=0 0 -0.175 rpy=1.5708 0 0

Commit message: 小改控制器

File: src/kuka_urdf/urdf/kuka_urdf.urdf (robot description, URDF)
Before this commit: robot kuka_urdf, 13 links, 12 joints
Links:
- link base_link: mass 72.8456791935468 -> 0.01
- link link1: mass 15.0345564818104 -> 0.01
- link link2: mass 13.9287847526223 -> 0.01
- link link3: mass 12.8506822129936 -> 0.01
- link link4: mass 2.38079247091277 -> 0.01
- link link5: mass 1.73398183318851 -> 0.01
- link link6: mass 0.21569146659832 -> 0.01
- link link7: mass 0.0603242087036552 -> 0.01
- link tabelLink1: mass 7.28336977784291 -> 0.01
- link tableEeffortLink: mass 3.48926224058707 -> 0.01
- link tableLink2: mass 0.32267569246235 -> 0.01
